Commit message: slam

File: xxu_nav_2026/src/xxu_description/urdf/plugins/gazebo_sensor_plugin.xacro (robot description, xacro)
@@ -8,10 +8,10 @@
     - <topic>      传感器数据通过 Gazebo Transport 发布到该 GZ 话题
     - <frame_id>   设置消息头中的坐标系（注意：Gazebo Harmonic 有一个 bug，
-                   会忽略 frame_id 标签，导致传感器始终附着在 odom_link 上）
+                   会忽略 frame_id 标签，导致传感器始终附着在模型根节点上）
     - <pose>       传感器相对于 reference_link 的位姿（x y z roll pitch yaw）
     - 需配合 ros_gz_bridge 的 parameter_bridge 将 GZ 话题桥接到 ROS 2 话题
   注意：
     由于 Gazebo Harmonic 的传感器放置 bug，即使指定了 reference_link，
-    传感器也会被放置到 TF 树的根节点（odom_link），且 frame_id 会被忽略。
+    传感器也会被放置到 TF 树的模型根节点，且 frame_id 会被忽略。
     因此在实际使用中，需要通过 frame_republisher（如 scan_frame_republisher.py）
     将 frame_id 修正为正确的坐标系（如 radar_link），并通过 ros_gz_bridge
@@ -50,5 +50,5 @@
     <!--
       Gazebo reference 标签：将传感器关联到指定的 link。
-      注意：Gazebo Harmonic 存在已知 bug，可能忽略此 reference，将传感器挂载到 odom_link。
+      注意：Gazebo Harmonic 存在已知 bug，可能忽略此 reference，将传感器挂载到模型根节点。
     -->
     <gazebo reference="${reference_link}">

File: xxu_nav_2026/src/xxu_description/urdf/xxu.urdf.xacro (robot description, xacro)
@@ -3,5 +3,6 @@
   <!--
     XXU 简化模型
-    TF 树：odom_link -> base_footprint -> base_link -> radar_link, wheel_fl, wheel_fr, wheel_rl, wheel_rr
+    静态 TF 树：base_link -> base_footprint, radar_link, wheel_fl, wheel_fr, wheel_rl, wheel_rr
+    动态 TF 树：odom -> base_link 由 Small Point-LIO 发布。
   -->
   <xacro:include filename="wheel.urdf.xacro"/>
@@ -89,9 +90,6 @@
     </link>
   </xacro:macro>
-  <!-- odom_link -->
-  <link name="odom_link"/>
   <!-- base_footprint：base_link 在地面的投影，轮子与地面保留 1 mm 缝隙 -->
   <link name="base_footprint"/>
-  <xacro:fixed_joint name="odom_joint" parent="odom_link" child="base_footprint"/>
   <!-- base_link -->
   <xacro:cylinder_link
@@ -104,5 +102,5 @@
     izz="${base_mass * base_radius * base_radius / 2}"
     material="chassis_blue"/>
-  <xacro:fixed_joint name="base_footprint_joint" parent="base_footprint" child="base_link" xyz="0 0 ${base_link_z}"/>
+  <xacro:fixed_joint name="base_footprint_joint" parent="base_link" child="base_footprint" xyz="0 0 ${-base_link_z}"/>
   <!-- radar_link -->
   <xacro:box_link

File: xxu_nav_2026/src/xxu_description/urdf/xxu_gazebo.urdf.xacro (robot description, xacro)
@@ -3,5 +3,6 @@
   <!--
     XXU Gazebo 仿真模型
-    TF 树：odom_link -> base_footprint -> base_link -> radar_link + 4 wheels (continuous joints)
+    静态 TF 树：base_link -> base_footprint, radar_link + 4 wheels (continuous joints)
+    动态 TF 树：odom -> base_link 由 Small Point-LIO 发布。
   -->
   <xacro:include filename="wheel.urdf.xacro"/>
@@ -98,8 +99,6 @@
     </link>
   </xacro:macro>
-  <!-- odom_link -->
-  <link name="odom_link"/>
+  <!-- base_footprint：base_link 在地面的投影。odom -> base_link 由 LIO 动态发布。 -->
   <link name="base_footprint"/>
-  <xacro:fixed_joint name="odom_joint" parent="odom_link" child="base_footprint"/>
   <!-- base_link -->
   <xacro:cylinder_link
@@ -112,5 +111,5 @@
     izz="${base_mass * base_radius * base_radius / 2}"
     material="chassis_blue"/>
-  <xacro:fixed_joint name="base_footprint_joint" parent="base_footprint" child="base_link" xyz="0 0 ${base_link_z}"/>
+  <xacro:fixed_joint name="base_footprint_joint" parent="base_link" child="base_footprint" xyz="0 0 ${-base_link_z}"/>
   <!-- radar_link: Mid-360 圆柱外形 -->
   <link name="radar_link">

Commit message: on COMPLETE mid_plugins

File: xxu_nav_2026/src/xxu_description/urdf/plugins/gazebo_sensor_plugin.xacro (robot description, xacro)
@@ -197,3 +197,40 @@
     </gazebo>
   </xacro:macro>
+  <!-- ====================================================================== -->
+  <!--             Livox MID-360 风格 Gazebo System 插件（原生射线点云）          -->
+  <!-- ====================================================================== -->
+  <!--
+    该插件挂在 reference_link 上，通过 Gazebo Physics RaycastData 生成非重复
+    MID-360 风格点云。它发布 Gazebo Transport PointCloudPacked，可由
+    ros_gz_bridge 桥接为 ROS 2 PointCloud2 后送入 Small Point-LIO。
+  -->
+  <xacro:macro
+    name="gazebo_mid360_livox_system_plugin"
+    params="
+      reference_link
+      topic:='/mid360/livox_points_gz'
+      frame_id:='radar_link'
+      update_rate:='10'
+      samples:='12000'
+      range_min:='0.1'
+      range_max:='40.0'
+      min_vertical:='-0.1221730'
+      max_vertical:='0.9075712'
+      sensor_pose:='0 0 0 0 0 0'">
+    <gazebo>
+      <plugin
+        filename="liblivox_mid360_system.so"
+        name="xxu_livox_sim::LivoxMid360System">
+        <topic>${topic}</topic>
+        <frame_id>${frame_id}</frame_id>
+        <update_rate>${update_rate}</update_rate>
+        <samples>${samples}</samples>
+        <range_min>${range_min}</range_min>
+        <range_max>${range_max}</range_max>
+        <min_vertical>${min_vertical}</min_vertical>
+        <max_vertical>${max_vertical}</max_vertical>
+        <sensor_pose>${sensor_pose}</sensor_pose>
+      </plugin>
+    </gazebo>
+  </xacro:macro>
 </robot>

File: xxu_nav_2026/src/xxu_description/urdf/xxu_gazebo.urdf.xacro (robot description, xacro)
@@ -10,4 +10,5 @@
   <xacro:include filename="plugins/gazebo_sensor_plugin.xacro"/>
   <xacro:arg name="controllers_file" default="src/xxu_description/config/xxu_ros2_control.yaml"/>
+  <xacro:arg name="use_livox_native" default="false"/>
   <!-- 尺寸和质量参数 -->
   <xacro:property name="base_radius" value="0.25"/>
@@ -174,4 +175,12 @@
     range_max="${mid360_range_max}"
     pose="0 0 ${radar_height / 2} 0 0 0"/>
+  <xacro:if value="$(arg use_livox_native)">
+    <xacro:gazebo_mid360_livox_system_plugin
+      reference_link="radar_link"
+      topic="/mid360/livox_points_gz"
+      frame_id="radar_link"
+      range_max="${mid360_range_max}"
+      sensor_pose="0.20565 0 0.1520 0 0.1745 0"/>
+  </xacro:if>
   <!-- 轮子物理属性 -->
   <gazebo reference="wheel_fl">

Commit message: lio完成

File: xxu_nav_2026/src/xxu_description/urdf/plugins/gazebo_sensor_plugin.xacro (robot description, xacro)
@@ -55,6 +55,6 @@
       <!-- sensor type="imu"：Gazebo 内置 IMU 传感器，输出角速度和线加速度 -->
       <sensor name="${sensor_name}" type="imu">
-        <!-- 传感器始终开启（1 = true），不随仿真暂停而关闭 -->
-        <always_on>1</always_on>
+        <!-- 传感器仅在仿真运行时更新（0 = false），避免暂停/初始化时产生异常时间戳 -->
+        <always_on>0</always_on>
         <!-- 传感器数据更新频率，单位 Hz -->
         <update_rate>${update_rate}</update_rate>
@@ -212,5 +212,6 @@
       frame_id:='radar_link'
       update_rate:='10'
-      samples:='12000'
+      samples:='2400'
+      rays_per_batch:='240'
       range_min:='0.1'
       range_max:='40.0'
@@ -222,8 +223,10 @@
         filename="liblivox_mid360_system.so"
         name="xxu_livox_sim::LivoxMid360System">
+        <reference_link>${reference_link}</reference_link>
         <topic>${topic}</topic>
         <frame_id>${frame_id}</frame_id>
         <update_rate>${update_rate}</update_rate>
         <samples>${samples}</samples>
+        <rays_per_batch>${rays_per_batch}</rays_per_batch>
         <range_min>${range_min}</range_min>
         <range_max>${range_max}</range_max>

File: xxu_nav_2026/src/xxu_description/urdf/xxu.urdf.xacro (robot description, xacro)
@@ -3,6 +3,6 @@
   <!--
     XXU 简化模型
-    静态 TF 树：base_link -> base_footprint, radar_link, wheel_fl, wheel_fr, wheel_rl, wheel_rr
-    动态 TF 树：odom -> base_link 由 Small Point-LIO 发布。
+    静态 TF 树：base_footprint -> base_link -> mid360_link, wheel_fl, wheel_fr, wheel_rl, wheel_rr
+    动态 TF 树：odom -> base_footprint 由 Small Point-LIO 发布。
   -->
   <xacro:include filename="wheel.urdf.xacro"/>
@@ -16,6 +16,6 @@
   <xacro:property name="radar_height" value="0.060"/>
   <xacro:property name="radar_size" value="${radar_length} ${radar_width} ${radar_height}"/>
-  <xacro:property name="radar_xyz" value="0.2 0 0.12"/>
-  <xacro:property name="radar_rpy" value="0 0.1745 0"/>
+  <xacro:property name="mid360_xyz" value="0.20565 0 0.1520"/>
+  <xacro:property name="mid360_rpy" value="0 0.1745 0"/>
   <xacro:property name="radar_mass" value="0.265"/>
   <!-- 全向轮参数 -->
@@ -90,5 +90,5 @@
     </link>
   </xacro:macro>
-  <!-- base_footprint：base_link 在地面的投影，轮子与地面保留 1 mm 缝隙 -->
+  <!-- base_footprint：地面投影原点，odom 直接连接到该帧。base_link 在其上方 -->
   <link name="base_footprint"/>
   <!-- base_link -->
@@ -102,8 +102,8 @@
     izz="${base_mass * base_radius * base_radius / 2}"
     material="chassis_blue"/>
-  <xacro:fixed_joint name="base_footprint_joint" parent="base_link" child="base_footprint" xyz="0 0 ${-base_link_z}"/>
-  <!-- radar_link -->
+  <xacro:fixed_joint name="base_footprint_joint" parent="base_footprint" child="base_link" xyz="0 0 ${base_link_z}"/>
+  <!-- mid360_link -->
   <xacro:box_link
-    name="radar_link"
+    name="mid360_link"
     size="${radar_size}"
     mass="${radar_mass}"
@@ -112,5 +112,5 @@
     izz="${radar_mass * (radar_length * radar_length + radar_width * radar_width) / 12}"
     material="radar_red"/>
-  <xacro:fixed_joint name="radar_joint" parent="base_link" child="radar_link" xyz="${radar_xyz}" rpy="${radar_rpy}"/>
+  <xacro:fixed_joint name="mid360_joint" parent="base_link" child="mid360_link" xyz="${mid360_xyz}" rpy="${mid360_rpy}"/>
   <!-- 四轮全向轮底盘，轮轴朝向 base_link 中心 -->
   <xacro:wheel name="wheel_fl" radius="${wheel_radius}" width="${wheel_width}" mass="${wheel_mass}"/>

File: xxu_nav_2026/src/xxu_description/urdf/xxu_gazebo.urdf.xacro (robot description, xacro)
@@ -3,6 +3,6 @@
   <!--
     XXU Gazebo 仿真模型
-    静态 TF 树：base_link -> base_footprint, radar_link + 4 wheels (continuous joints)
-    动态 TF 树：odom -> base_link 由 Small Point-LIO 发布。
+    静态 TF 树：base_footprint -> base_link -> mid360_link + 4 wheels (continuous joints)
+    动态 TF 树：odom -> base_footprint 由 Small Point-LIO 发布。
   -->
   <xacro:include filename="wheel.urdf.xacro"/>
@@ -17,6 +17,6 @@
   <xacro:property name="radar_radius" value="0.0325"/>
   <xacro:property name="radar_height" value="0.065"/>
-  <xacro:property name="radar_xyz" value="0.2 0 0.12"/>
-  <xacro:property name="radar_rpy" value="0 0.1745 0"/>
+  <xacro:property name="mid360_xyz" value="0.20565 0 0.1520"/>
+  <xacro:property name="mid360_rpy" value="0 0.1745 0"/>
   <xacro:property name="radar_mass" value="0.265"/>
   <xacro:property name="mid360_range_max" value="40.0"/>
@@ -100,5 +100,5 @@
     </link>
   </xacro:macro>
-  <!-- base_footprint：base_link 在地面的投影。odom -> base_link 由 LIO 动态发布。 -->
+  <!-- base_footprint：地面投影原点。odom -> base_footprint 由 LIO 动态发布，base_link 在其上方。 -->
   <link name="base_footprint"/>
   <!-- base_link -->
@@ -112,9 +112,9 @@
     izz="${base_mass * base_radius * base_radius / 2}"
     material="chassis_blue"/>
-  <xacro:fixed_joint name="base_footprint_joint" parent="base_link" child="base_footprint" xyz="0 0 ${-base_link_z}"/>
-  <!-- radar_link: Mid-360 圆柱外形 -->
-  <link name="radar_link">
+  <xacro:fixed_joint name="base_footprint_joint" parent="base_footprint" child="base_link" xyz="0 0 ${base_link_z}"/>
+  <!-- mid360_link: LiDAR and IMU measurement frame. -->
+  <link name="mid360_link">
     <visual>
-      <origin xyz="0 0 0" rpy="0 0 0"/>
+      <origin xyz="0 0 ${-radar_height / 2}" rpy="0 0 0"/>
       <geometry>
         <cylinder radius="${radar_radius}" length="${radar_height}"/>
@@ -124,5 +124,5 @@
     <!-- 顶部半球，模仿 Mid-360 外观 -->
     <visual>
-      <origin xyz="0 0 ${radar_height / 2}" rpy="0 0 0"/>
+      <origin xyz="0 0 0" rpy="0 0 0"/>
       <geometry>
         <sphere radius="${radar_radius}"/>
@@ -131,5 +131,5 @@
     </visual>
     <collision>
-      <origin xyz="0 0 0" rpy="0 0 0"/>
+      <origin xyz="0 0 ${-radar_height / 2}" rpy="0 0 0"/>
       <geometry>
         <cylinder radius="${radar_radius}" length="${radar_height}"/>
@@ -147,5 +147,5 @@
     </inertial>
   </link>
-  <xacro:fixed_joint name="radar_joint" parent="base_link" child="radar_link" xyz="${radar_xyz}" rpy="${radar_rpy}"/>
+  <xacro:fixed_joint name="mid360_joint" parent="base_link" child="mid360_link" xyz="${mid360_xyz}" rpy="${mid360_rpy}"/>
   <!-- 四轮全向轮底盘（连续关节） -->
   <xacro:wheel name="wheel_fl" radius="${wheel_radius}" width="${wheel_width}" mass="${wheel_mass}"/>
@@ -168,18 +168,20 @@
     wheel_radius="${wheel_radius}"
     controllers_file="$(arg controllers_file)"/>
-  <xacro:gazebo_imu_plugin reference_link="radar_link" frame_id="radar_link"/>
-  <xacro:gazebo_mid360_lidar_plugin
-    reference_link="radar_link"
-    topic="/mid360"
-    frame_id="radar_link"
-    range_max="${mid360_range_max}"
-    pose="0 0 ${radar_height / 2} 0 0 0"/>
+  <xacro:gazebo_imu_plugin reference_link="base_footprint" frame_id="base_footprint"/>
+  <xacro:unless value="$(arg use_livox_native)">
+    <xacro:gazebo_mid360_lidar_plugin
+      reference_link="base_footprint"
+      topic="/mid360"
+      frame_id="base_footprint"
+      range_max="${mid360_range_max}"
+      pose="0 0 0 0 0 0"/>
+  </xacro:unless>
   <xacro:if value="$(arg use_livox_native)">
     <xacro:gazebo_mid360_livox_system_plugin
-      reference_link="radar_link"
+      reference_link="base_footprint"
       topic="/mid360/livox_points_gz"
-      frame_id="radar_link"
+      frame_id="base_footprint"
       range_max="${mid360_range_max}"
-      sensor_pose="0.20565 0 0.1520 0 0.1745 0"/>
+      sensor_pose="0 0 0 0 0 0"/>
   </xacro:if>
   <!-- 轮子物理属性 -->
